Commit message: initial changes

File: l_hand.urdf (robot description, URDF)
Before this commit: robot l_hand, 8 links, 7 joints
Links:
- added link l_lil2, mass 0.010; collision mesh filename=file:///home/yeshi/icub-gazebo/icub/meshes/collision/l_hand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; visual mesh filename=file:///home/yeshi/icub-gazebo/icub/meshes/visual/l_hand/l_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
- link l_hand_base_link: geometry collision mesh filename=file:///home/yeshi/icub-gazebo/icub/meshes/collision/l_hand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; collision mesh filename=file:///home/yeshi/icub-gazebo/icub/meshes/collision/l_hand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
Joints:
- added joint l_lij4: type revolute, parent l_lil1, child l_lil2, origin xyz=0.0148 0 0 rpy=1.5708 0 0, axis 0.087189 0.017426 0.996039, limit lower=0 upper=1.5708 effort=10 velocity=0.5
- joint l_aij3: origin xyz=0.01225 -0.075498 -0.027259 rpy=0.0959 0.017493 -1.57079 -> xyz=0.012 0 0 rpy=1.5708 0 0
- joint l_aij4: origin xyz=0.03 0 0 rpy=0 0 0 -> xyz=0.0259 0 0 rpy=0 0 0
- joint l_aij5: origin xyz=0.03 0 0 rpy=0 0 0 -> xyz=0.022 0 0 rpy=0 0 0
- joint l_aij6: origin xyz=0 0 0 rpy=0 0 0 -> xyz=0.01225 -0.0643 -0.027 rpy=-1.4749 -0.072507 -1.57079
- joint l_lij3: origin xyz=0 0 0 rpy=0 0 0 -> xyz=0.0148 0 0 rpy=1.5708 0 0
