Commit message: hands base links name changed to convention

File: both_hands.urdf (robot description, URDF)
Before this commit: robot both_hands, 43 links, 42 joints
Links:
- removed link l_hand_base_link
- removed link r_hand_base_link
- added link l_hand, mass 0.010; collision mesh filename=file:///home/yeshi/icub-gazebo/icub/meshes/collision/l_hand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; collision mesh filename=file:///home/yeshi/icub-gazebo/icub/meshes/collision/l_hand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
- added link r_hand, mass 0.010; collision mesh filename=file:///home/yeshi/icub-gazebo/icub/meshes/collision/r_hand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; collision mesh filename=file:///home/yeshi/icub-gazebo/icub/meshes/collision/r_hand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
Joints:
- joint l_aij6: parent l_hand_base_link -> l_hand
- joint l_lij6: parent l_hand_base_link -> l_hand
- joint l_mj6: parent l_hand_base_link -> l_hand
- joint l_rij6: parent l_hand_base_link -> l_hand
- joint l_tj2: parent l_hand_base_link -> l_hand
- joint left_base_fixed_joint: child l_hand_base_link -> l_hand
- joint r_aij6: parent r_hand_base_link -> r_hand
- joint r_lij6: parent r_hand_base_link -> r_hand
- joint r_mj6: parent r_hand_base_link -> r_hand
- joint r_rij6: parent r_hand_base_link -> r_hand
- joint r_tj2: parent r_hand_base_link -> r_hand
- joint right_base_fixed_joint: child r_hand_base_link -> r_hand

Commit message: palm dh frames added

File: both_hands.urdf (robot description, URDF)
Before this commit: robot both_hands, 43 links, 42 joints
Links:
- added link l_hand_dh_frame, mass 0
- added link r_hand_dh_frame, mass 0
Joints:
- added joint l_hand_dh_frame_fixed_joint: type fixed, parent l_hand, child l_hand_dh_frame, origin xyz=0 -0.04 0 rpy=0 -0 0, axis 0 0 0
- added joint r_hand_dh_frame_fixed_joint: type fixed, parent r_hand, child r_hand_dh_frame, origin xyz=0 -0.04 0 rpy=0 -0 0, axis 0 0 0
