Commit message: proper representation achieved

File: l_hand_mine.urdf (robot description, URDF)
Before this commit: robot l_hand_mine, 22 links, 21 joints
Joints:
- joint l_aij6: origin xyz=0.01225 -0.0643 -0.027 rpy=-1.4749 -0.072507 -1.57079 -> xyz=0.01225 -0.0643 -0.027 rpy=-1.4749 0.017507 -1.57079
- joint l_tj6: origin xyz=0.022 0 0 rpy=1.5708 0 0 -> xyz=0.022 0 0 rpy=0 0 0

Commit message: ring and little finger last joint axis of rotation corrected

File: l_hand_mine.urdf (robot description, URDF)
Before this commit: robot l_hand_mine, 22 links, 21 joints
Joints:
- joint l_lij5: origin xyz=0.02 0 -0.00385 rpy=1.5708 0 0 -> xyz=0.02 0 -0.00385 rpy=0 0 0
- joint l_rij5: origin xyz=0.0242 0 0.0045 rpy=1.5708 0 0 -> xyz=0.0242 0 0.0045 rpy=0 0 0

Commit message: left hand fine tuned

File: l_hand_mine.urdf (robot description, URDF)
Before this commit: robot l_hand_mine, 22 links, 21 joints
Links:
- link l_hand_base_link: geometry collision mesh filename=file:///home/yeshi/icub-gazebo/icub/meshes/collision/l_hand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; collision mesh filename=file:///home/yeshi/icub-gazebo/icub/meshes/collision/l_hand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

Commit message: hands base link name changed

File: l_hand_mine.urdf (robot description, URDF)
Before this commit: robot l_hand_mine, 22 links, 21 joints
Links:
- removed link l_hand_base_link
- added link l_hand, mass 0.010; collision mesh filename=file:///home/yeshi/icub-gazebo/icub/meshes/collision/l_hand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; collision mesh filename=file:///home/yeshi/icub-gazebo/icub/meshes/collision/l_hand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
Joints:
- joint base_fixed_joint: child l_hand_base_link -> l_hand
- joint l_aij6: parent l_hand_base_link -> l_hand
- joint l_lij6: parent l_hand_base_link -> l_hand
- joint l_mj6: parent l_hand_base_link -> l_hand
- joint l_rij6: parent l_hand_base_link -> l_hand
- joint l_tj2: parent l_hand_base_link -> l_hand

File: r_hand_mine.urdf (robot description, URDF)
Before this commit: robot r_hand_mine, 22 links, 21 joints
Links:
- removed link r_hand_base_link
- added link r_hand, mass 0.010; collision mesh filename=file:///home/yeshi/icub-gazebo/icub/meshes/collision/r_hand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; collision mesh filename=file:///home/yeshi/icub-gazebo/icub/meshes/collision/r_hand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
Joints:
- joint base_fixed_joint: child r_hand_base_link -> r_hand
- joint r_aij6: parent r_hand_base_link -> r_hand
- joint r_lij6: parent r_hand_base_link -> r_hand
- joint r_mj6: parent r_hand_base_link -> r_hand
- joint r_rij6: parent r_hand_base_link -> r_hand
- joint r_tj2: parent r_hand_base_link -> r_hand

Commit message: palm dh frame added

File: l_hand_mine.urdf (robot description, URDF)
Before this commit: robot l_hand_mine, 22 links, 21 joints
Links:
- added link l_hand_dh_frame, mass 0
Joints:
- added joint l_hand_dh_frame_fixed_joint: type fixed, parent l_hand, child l_hand_dh_frame, origin xyz=0 -0.04 0 rpy=0 -0 0, axis 0 0 0
